File: EPROMAdapter.sch (EAGLE design)
At the start: 1 part

Commit message: wrapped that up
Parts:
- added 2513: 2513-CHARACTER, memory:2513-CHARACTER
- renumbered EPROM to 2716
Connections:
- new net !CE: 2513.!CE, 2716A.!CE, 2716A.!OE
- new net A0: 2513.A1, 2716A.A0
- new net A1: 2513.A2, 2716A.A1
- new net A2: 2513.A3, 2716A.A2
- new net A3: 2513.A4, 2716A.A3
- new net A4: 2513.A5, 2716A.A4
- new net A5: 2513.A6, 2716A.A5
- new net A6: 2513.A7, 2716A.A6
- new net A7: 2513.A8, 2716A.A7
- new net A8: 2513.A9, 2716A.A8
- new net D1: 2513.O1, 2716A.O0
- new net D2: 2513.O2, 2716A.O1
- new net D3: 2513.O3, 2716A.O2
- new net D4: 2513.O4, 2716A.O3
- new net D5: 2513.O5, 2716A.O4
- new net GND: 2513.GND, 2716A.A10, 2716A.A9, 2716P.GND
- new net VCC: 2513.VCC, 2716P.VCC
